File: 0504/0504.kicad_pcb (KiCad board)
At the start: 2 copper layers, 11 parts, among them J1 Conn_01x01_Socket, J2 Conn_01x01_Socket, U1 LM2577T-ADJ_NOPB

Commit message: Version cambiada y corregida
Parts:
- removed J2: Conn_01x01_Socket, Connector_Wire:SolderWire-0.5sqmm_1x02_P4.6mm_D0.9mm_OD2.1mm
- added J3: Conn_01x02_Pin, Connector_Wire:SolderWire-0.5sqmm_1x02_P4.6mm_D0.9mm_OD2.1mm, F.Cu at (86.5, 82.0)
- J1: value Conn_01x01_Socket -> Conn_01x02_Pin
- moved L1 52.7 mm to (90.5, 73.5), turned to 0 degrees
- moved C1 44.5 mm to (91.0, 85.5), turned to -90 degrees
- moved U1 32.8 mm to (95.5, 90.5), turned to 90 degrees
- moved J1 25.4 mm to (122.5, 73.9), turned to -90 degrees
- moved R3 24.3 mm to (106.5, 80.0), turned to 180 degrees
- moved D1 23.6 mm to (114.5, 73.5), turned to 180 degrees
- moved R2 23.3 mm to (106.5, 85.5), turned to 0 degrees
- moved C3 22.0 mm to (116.0, 80.0)
- moved R1 21.1 mm to (106.5, 90.0)
- moved C2 20.8 mm to (116.0, 84.5)
Connections:
- J1 pad 2: (no net) -> GND
Routing:
- net Net-(D1-A): track 61.0 -> 22.4 mm
- net GND: track 36.0 -> 62.9 mm
- net (no net): track 26.6 -> 0.00 mm
- net Net-(U1-FEEDBACK): track 31.1 -> 15.5 mm
- net Net-(J3-Pin_1): track 30.5 -> 19.5 mm
- net Net-(C2-Pad1): track 6.23 -> 10.4 mm
- net Net-(U1-COMP): track 6.87 -> 8.81 mm
Other:
- board outline added: 44 x 27.5 mm
